File: hardware/strava-distance-display.sch (KiCad schematic (older format))
At the start: 12 parts, among them J1 Display, J2 Battery, J3 FTDI_CONN, SW1 reset, SW2 prog enable, U1 ESP-12F, U2 LD1117S33TR_SOT223

Commit message: Schematic now uses built-in KiCad's ESP-12F symbol + footprint.
And all the related error fixes as well..
Parts:
- removed U1: ESP-12F, RF_Modules:ESP-12E, symbol ESP-12F
- added R2: 10K, Resistors_SMD:R_0805_HandSoldering, symbol R
- added U1: ESP-12E, RF_Modules:ESP-12E, symbol ESP-12E
- C1: symbol C -> C-RESCUE-strava-distance-display
- R1: symbol R -> R-RESCUE-strava-distance-display
- U2: footprint TO_SOT_Packages_SMD:SOT-223-3_TabPin2 -> TO_SOT_Packages_SMD:SOT-223
Connections:
- wire segments 54 -> 41
Other:
- moved on the sheet: C1, C2, C4, C5, J1, J2, J3, R1, SW1, SW2, U2
